File: cad/stone_pcb_v1.kicad_sch (KiCad schematic)
At the start: 19 parts, among them J2 DRV8833, J3 DCDC-6V, J4 DCDC-5V, J5 USB_C_Receptacle_USB2.0_14P, J6 S2-Mini, J7 Breakouts, J8 S2-Mini, J9 Conn_01x02_Socket EXT_5V & GND, SW1 SW_SPST

Commit message: modified pcb
Parts:
- J1, J2: footprint Connector_PinHeader_2.54mm:PinHeader_1x06_P2.54mm_Vertical -> Connector_PinSocket_2.54mm:PinSocket_1x06_P2.54mm_Vertical
- J3, J4: footprint Connector_PinHeader_2.54mm:PinHeader_1x02_P2.54mm_Vertical -> Connector_PinSocket_2.54mm:PinSocket_1x02_P2.54mm_Vertical
- J6, J8: footprint Connector_PinHeader_2.54mm:PinHeader_1x08_P2.54mm_Horizontal -> Connector_PinSocket_2.54mm:PinSocket_1x08_P2.54mm_Vertical
- J7: footprint Connector_PinHeader_2.54mm:PinHeader_1x07_P2.54mm_Horizontal -> Connector_PinSocket_2.54mm:PinSocket_1x08_P2.54mm_Vertical
- J9: footprint Connector_PinHeader_2.54mm:PinHeader_1x01_P2.54mm_Horizontal -> Connector_PinSocket_2.54mm:PinSocket_1x02_P2.54mm_Vertical
Changed lines of the file:
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@@
 			)
 		)
-		(property "Footprint" "Connector_PinHeader_2.54mm:PinHeader_1x06_P2.54mm_Vertical"
+		(property "Footprint" "Connector_PinSocket_2.54mm:PinSocket_1x06_P2.54mm_Vertical"
 			(at 179.07 119.38 0)
 			(effects
@@
 			)
 		)
-		(property "Footprint" "Connector_PinHeader_2.54mm:PinHeader_1x01_P2.54mm_Horizontal"
+		(property "Footprint" "Connector_PinSocket_2.54mm:PinSocket_1x02_P2.54mm_Vertical"
 			(at 92.71 41.91 0)
 			(effects
@@
 			)
 		)
-		(property "Footprint" "Connector_PinHeader_2.54mm:PinHeader_1x08_P2.54mm_Horizontal"
+		(property "Footprint" "Connector_PinSocket_2.54mm:PinSocket_1x08_P2.54mm_Vertical"
 			(at 86.36 119.38 0)
 			(effects
@@
 			)
 		)
-		(property "Footprint" "Connector_PinHeader_2.54mm:PinHeader_1x08_P2.54mm_Horizontal"
+		(property "Footprint" "Connector_PinSocket_2.54mm:PinSocket_1x08_P2.54mm_Vertical"
 			(at 114.3 121.92 0)
 			(effects
@@
 			)
 		)
-		(property "Footprint" "Connector_PinHeader_2.54mm:PinHeader_1x02_P2.54mm_Vertical"
+		(property "Footprint" "Connector_PinSocket_2.54mm:PinSocket_1x02_P2.54mm_Vertical"
 			(at 149.86 66.04 0)
 			(effects
@@
 			)
 		)
-		(property "Footprint" "Connector_PinHeader_2.54mm:PinHeader_1x02_P2.54mm_Vertical"
+		(property "Footprint" "Connector_PinSocket_2.54mm:PinSocket_1x02_P2.54mm_Vertical"
 			(at 172.72 66.04 0)
 			(effects
@@
 			)
 		)
-		(property "Footprint" "Connector_PinHeader_2.54mm:PinHeader_1x07_P2.54mm_Horizontal"
+		(property "Footprint" "Connector_PinSocket_2.54mm:PinSocket_1x08_P2.54mm_Vertical"
 			(at 46.99 121.92 0)
 			(effects
@@
 			)
 		)
-		(property "Footprint" "Connector_PinHeader_2.54mm:PinHeader_1x06_P2.54mm_Vertical"
+		(property "Footprint" "Connector_PinSocket_2.54mm:PinSocket_1x06_P2.54mm_Vertical"
 			(at 153.67 119.38 0)
 			(effects

Commit message: finished pcb design
Parts:
- removed J3: DCDC-6V, Connector_PinSocket_2.54mm:PinSocket_1x02_P2.54mm_Vertical, symbol Connector:Conn_01x02_Socket
- removed J4: DCDC-5V, Connector_PinSocket_2.54mm:PinSocket_1x02_P2.54mm_Vertical, symbol Connector:Conn_01x02_Socket
- removed SW1: SW_SPST, TestPoint:TestPoint_Pad_D2.0mm, symbol Switch:SW_SPST
- added J10: Conn_01x02_Socket 5V & GND CAMLINE, Connector_PinSocket_2.54mm:PinSocket_1x02_P2.54mm_Vertical, symbol Connector:Conn_01x02_Socket
- added TP6: TP VBUS, TestPoint:TestPoint_Pad_D2.0mm, symbol Connector:TestPoint
- added TP7: Switch1, TestPoint:TestPoint_Pad_D2.0mm, symbol Connector:TestPoint
- added TP8: Switch2, TestPoint:TestPoint_Pad_D2.0mm, symbol Connector:TestPoint
- J7: footprint Connector_PinSocket_2.54mm:PinSocket_1x08_P2.54mm_Vertical -> Connector_PinSocket_2.54mm:PinSocket_1x07_P2.54mm_Vertical
Connections:
- net at J1.1 (Pin_1): now also J8.7 (Pin_7); no longer J8.8 (Pin_8)
- net GND: now reaches 5.1k1.1, 5.1k2.1, D1.1 (K), J2.4 (Pin_4), J5.A1 (GND), J5.A12 (GND), J5.B1 (GND), J5.B12 (GND), J5.S1 (SHIELD), J6.2 (Pin_2), J7.7 (Pin_7), J9.1 (Pin_1), TP5.1
- net GND: now also J10.2 (Pin_2)
- net VBUS: now reaches J5.A4 (VBUS), J5.A9 (VBUS), J5.B4 (VBUS), J5.B9 (VBUS), J9.2 (Pin_2)
- net VBUS: now also TP7.1; no longer J6.1 (Pin_1)
- net at J8.5 (Pin_5): now also J2.2 (Pin_2)
- net at J8.6 (Pin_6): now also J2.1 (Pin_1); no longer J2.2 (Pin_2)
- net at R2.2: now also J2.3 (Pin_3), J6.1 (Pin_1), J10.1 (Pin_1), TP6.1, TP8.1
Other:
- moved on the sheet: D1, R2, TP5
