File: cad/stone_pcb_v1.kicad_pcb (KiCad board)
At the start: 2 copper layers, 19 parts, among them J2 DRV8833, J3 DCDC-6V, J4 DCDC-5V, J5 USB_C_Receptacle_USB2.0_14P, J6 S2-Mini, J7 Breakouts, J8 S2-Mini, J9 Conn_01x02_Socket EXT_5V & GND, SW1 SW_SPST

Commit message: modified pcb
Parts:
- J1, J2: footprint Connector_PinHeader_2.54mm:PinHeader_1x06_P2.54mm_Vertical -> Connector_PinSocket_2.54mm:PinSocket_1x06_P2.54mm_Vertical
- J3, J4: footprint Connector_PinHeader_2.54mm:PinHeader_1x02_P2.54mm_Vertical -> Connector_PinSocket_2.54mm:PinSocket_1x02_P2.54mm_Vertical
- J6, J8: footprint Connector_PinHeader_2.54mm:PinHeader_1x08_P2.54mm_Horizontal -> Connector_PinSocket_2.54mm:PinSocket_1x08_P2.54mm_Vertical
- J7: footprint Connector_PinHeader_2.54mm:PinHeader_1x07_P2.54mm_Horizontal -> Connector_PinSocket_2.54mm:PinSocket_1x08_P2.54mm_Vertical
- J9: footprint Connector_PinHeader_2.54mm:PinHeader_1x01_P2.54mm_Horizontal -> Connector_PinSocket_2.54mm:PinSocket_1x02_P2.54mm_Vertical
- moved D1 83.0 mm to (62.5, 38.0)
- moved SW1 81.2 mm to (160.0, 27.5)
- moved TP5 73.8 mm to (160.0, 34.0)
- moved J4 73.0 mm to (141.0, 28.0)
- moved R2 70.7 mm to (73.5, 38.0)
- moved J3 69.8 mm to (129.5, 28.2)
- moved J5 63.7 mm to (64.5, 49.8), turned to -90 degrees
- moved 5.1k1 60.5 mm to (61.5, 60.0)
- moved 5.1k2 59.2 mm to (61.5, 66.0)
- moved TP1 50.2 mm to (132.0, 48.0)
- moved TP2 40.8 mm to (132.0, 52.8)
- moved TP3 40.2 mm to (132.0, 57.7)
- moved TP4 30.9 mm to (132.0, 62.5)
- moved J7 29.7 mm to (93.1, 71.0), turned to -90 degrees
- moved J1 25.3 mm to (110.0, 61.2), turned to 180 degrees
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
Commit message: changes to pcb
Parts:
- moved SW1 43.5 mm to (116.5, 28.5)
- moved TP5 43.5 mm to (116.5, 35.0)
- moved J3 39.5 mm to (90.0, 29.2)
- moved J4 39.5 mm to (101.5, 29.0)
- moved TP1 15.5 mm to (116.5, 48.0)
- moved TP2 15.5 mm to (116.5, 52.8)
- moved TP3 15.5 mm to (116.5, 57.7)
- moved TP4 15.5 mm to (116.5, 62.5)
Changed lines of the file:
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@@
 			(psa4output no)
 			(plot_black_and_white yes)
-			(plotinvisibletext no)
 			(sketchpadsonfab no)
 			(plotpadnumbers no)
@@
 	(footprint "TestPoint:TestPoint_Pad_D2.0mm"
 		(layer "F.Cu")
-		(at 132 57.666667)
+		(at 116.5 57.666667)
 		(descr "SMD pad as test Point, diameter 2.0mm")
 		(tags "test point SMD pad")
@@
 	(footprint "TestPoint:TestPoint_Pad_D2.0mm"
 		(layer "F.Cu")
-		(at 132 62.5)
+		(at 116.5 62.5)
 		(descr "SMD pad as test Point, diameter 2.0mm")
 		(tags "test point SMD pad")
@@
 	(footprint "TestPoint:TestPoint_Pad_D2.0mm"
 		(layer "F.Cu")
-		(at 132 48)
+		(at 116.5 48)
 		(descr "SMD pad as test Point, diameter 2.0mm")
 		(tags "test point SMD pad")
@@
 	(footprint "TestPoint:TestPoint_Pad_D2.0mm"
 		(layer "F.Cu")
-		(at 132 52.833333)
+		(at 116.5 52.833333)
 		(descr "SMD pad as test Point, diameter 2.0mm")
 		(tags "test point SMD pad")
@@
 	(footprint "TestPoint:TestPoint_Pad_D2.0mm"
 		(layer "F.Cu")
-		(at 160 27.5)
+		(at 116.5 28.525)
 		(descr "SMD pad as test Point, diameter 2.0mm")
 		(tags "test point SMD pad")
@@
 	(footprint "TestPoint:TestPoint_Pad_D2.0mm"
 		(layer "F.Cu")
-		(at 160 34)
+		(at 116.5 35.025)
 		(descr "SMD pad as test Point, diameter 2.0mm")
 		(tags "test point SMD pad")
@@
 	(footprint "Connector_PinSocket_2.54mm:PinSocket_1x02_P2.54mm_Vertical"
 		(layer "F.Cu")
-		(at 129.5 28.225)
+		(at 90.025 29.25)
 		(descr "Through hole straight socket strip, 1x02, 2.54mm pitch, single row (from Kicad 4.0.7), script generated")
 		(tags "Through hole socket strip THT 1x02 2.54mm single row")
@@
 	(footprint "Connector_PinSocket_2.54mm:PinSocket_1x02_P2.54mm_Vertical"
 		(layer "F.Cu")
-		(at 141 27.96)
+		(at 101.525 28.985)
 		(descr "Through hole straight socket strip, 1x02, 2.54mm pitch, single row (from Kicad 4.0.7), script generated")
 		(tags "Through hole socket strip THT 1x02 2.54mm single row")

Commit message: finished pcb design
Parts:
- removed J3: DCDC-6V, Connector_PinSocket_2.54mm:PinSocket_1x02_P2.54mm_Vertical
- removed J4: DCDC-5V, Connector_PinSocket_2.54mm:PinSocket_1x02_P2.54mm_Vertical
- removed SW1: SW_SPST, TestPoint:TestPoint_Pad_D2.0mm
- added J10: Conn_01x02_Socket 5V & GND CAMLINE, Connector_PinSocket_2.54mm:PinSocket_1x02_P2.54mm_Vertical, F.Cu at (106.5, 39.5)
- added TP6: TP VBUS, TestPoint:TestPoint_Pad_D2.0mm, F.Cu at (98.5, 39.5)
- added TP7: Switch1, TestPoint:TestPoint_Pad_D2.0mm, F.Cu at (70.0, 39.5)
- added TP8: Switch2, TestPoint:TestPoint_Pad_D2.0mm, F.Cu at (73.5, 39.5)
- J7: footprint Connector_PinSocket_2.54mm:PinSocket_1x08_P2.54mm_Vertical -> Connector_PinSocket_2.54mm:PinSocket_1x07_P2.54mm_Vertical
- moved J9 56.2 mm to (63.2, 39.5), turned to 90 degrees
- moved D1 31.7 mm to (66.0, 69.5), turned to 180 degrees
- moved R2 28.4 mm to (62.2, 64.0)
- moved J8 20.7 mm to (99.4, 62.0), turned to 180 degrees
- moved TP1 18.8 mm to (128.5, 62.5)
- moved TP4 17.7 mm to (128.5, 49.5)
- moved J1 17.1 mm to (122.4, 49.5), turned to 0 degrees
- moved TP5 15.1 mm to (102.0, 39.5)
- moved J2 13.8 mm to (106.9, 49.5), turned to 0 degrees
- moved TP2 13.3 mm to (128.5, 58.5)
- moved J7 12.7 mm to (80.4, 70.0), turned to 90 degrees
- moved TP3 12.6 mm to (128.5, 53.8)
- moved 5.1k2 5.05 mm to (62.2, 61.0)
- moved 5.1k1 2.12 mm to (62.2, 58.0)
- moved J6 1.20 mm to (76.9, 44.3)
Connections:
- net Net-(D1-K) renamed /GND
- J2 pad 3: Net-(J2-Pin_3) -> Net-(J10-Pin_1)
- J5 pad A4: Net-(J6-Pin_1) -> /VBUS
- J5 pad A9: Net-(J6-Pin_1) -> /VBUS
- J5 pad B4: Net-(J6-Pin_1) -> /VBUS
- J5 pad B9: Net-(J6-Pin_1) -> /VBUS
- J6 pad 1: Net-(J6-Pin_1) -> Net-(J10-Pin_1)
- J8 pad 5: unconnected-(J8-Pin_5-Pad5) -> Net-(J2-Pin_2)
- J8 pad 6: Net-(J2-Pin_2) -> Net-(J2-Pin_1)
- J8 pad 7: Net-(J2-Pin_1) -> Net-(J1-Pin_1)
- J8 pad 8: Net-(J1-Pin_1) -> unconnected-(J8-Pin_8-Pad8)
- J9 pad 2: Net-(J6-Pin_1) -> /VBUS
- R2 pad 2: Net-(J4-Pin_1) -> Net-(J10-Pin_1)
Routing:
- net Net-(J10-Pin_1): track 0.00 -> 82.2 mm
- net Net-(J6-Pin_3): track 0.00 -> 27.5 mm
- net Net-(J1-Pin_1): track 0.00 -> 24.1 mm
- net Net-(J1-Pin_6): track 0.00 -> 24.1 mm
- net Net-(J6-Pin_4): track 0.00 -> 23.9 mm
- net /VBUS: track 0.00 -> 20.8 mm
- net Net-(J6-Pin_5): track 0.00 -> 20.3 mm
- net Net-(J6-Pin_6): track 0.00 -> 16.8 mm
- net Net-(J5-CC1): track 0.00 -> 15.3 mm, vias 0 -> 1
- net Net-(J6-Pin_7): track 0.00 -> 13.2 mm
- net Net-(J5-CC2): track 0.00 -> 10.5 mm
- net Net-(J2-Pin_6): track 0.00 -> 9.70 mm
- net Net-(J2-Pin_5): track 0.00 -> 9.70 mm
- net Net-(J6-Pin_8): track 0.00 -> 9.40 mm
- net Net-(J2-Pin_2): track 0.00 -> 7.57 mm
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- added copper zone on B.Cu, net /GND
Other:
- board outline added: 70.4 x 38.9 mm
- board text added: "-"
- board text added: "16"
- board text added: "18"
- board text added: "33"
- board text added: "35"
- board text added: "37"
- board text added: "39"
- board text added: "5.1k"
- board text added: "GND"
- board text added: "designed by prt"
- board text added: "still as stone"

Commit message: updated pcb
Routing:
- net Net-(J5-CC1): track 15.3 -> 15.9 mm, vias 1 -> 0
- added copper zone on F.Cu, net /GND
Changed lines of the file:
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@@
 			(psa4output no)
 			(plot_black_and_white yes)
+			(plotinvisibletext no)
 			(sketchpadsonfab no)
 			(plotpadnumbers no)
@@
 			"AAAAAAAAAAAAAAAAAAAAAAAAAAAAAAAAAAAAAAAAAAAAAAAAAAAAAAAAAAAAAAAAAAAAAAAAAAAA"
 			"AAAAAAAAAAAAAAAAAAAAAAAAAAAAAAAAAAAAAAAAAAAAAAAAAAAAAAAAAAAAAAAAAAAAAAAAAAAA"
+			"AAAAAAAAAAAAAAAAAAAAAAAAAAAAAAAAAAAAAAAAAAAAAAAAAAAAAAAAAAAAAAAAAAAAAAAAAAAA"
+			"AAAAAAAAAAAAAAAAAAAAAAAAAAAAAAAAAAAAAAAAAAAAAAAAAAAAAAAAAAAAAAAAAAAAAAAAAAAA"
+			"AAAAAAAAAAAAAAAAAAAAAAAAAAAAAAAAAAAAAAAAAAAAAAAAAAAAAAAAAAAAAAAAAAAAAAAAAAAA"
+			"AAAAAAAAAAAAAAAAAAAAAAAAAAAAAAAAAAAAAAAAAAAAAAAAAAAAAAAAAAAAAAAAAAAAAAAAAAAA"
+			"AAAAAAAAAAAAAAAAAAAAAAAAAAAAAAAAAAAAAAAAAAAAAAAAAAAAAAAAAAAAAAAAAAAAAAAAAAAA"
+			"AAAAAAAAAAAAAAAAAAAAAAAAAAAAAAAAAAAAAAAAAAAAAAAAAAAAAAAAAAAAAAAAAAAAAAAAAAAA"
+			"AAAAAAAAAAAAAAAAAAAAAAAAAAAAAAAAAAAAAAAAAAAAAAAAAAAAAAAAAAAAAAAAAAAAAAAAAAAA"
+			"AAAAAAAAAAAAAAAAAAAAAAAAAAAAAAAAAAAAAAAAAAAAAAAAAAAAAAAAAAAAAAAAAAAAAAAAAAAA"
+			"AAAAAAAAAAAAAAAAAAAAAAAAAAAAAAAAAAAAAAAAAAAAAAAAAAAAAAAAAAAAAAAAAAAAAAAAAAAA"
+			"AAAAAAAAAAAAAAAAAAAAAAAAAAAAAAAAAAAAAAAAAAAAAAAAAAAAAAAAAAAAAAAAAAAAAAAAAAAA"
+			"AAAAAAAAAAAAAAAAAAAAAAAAAAAAAAAAAAAAAAAAAAAAAAAAAAAAAAAAAAAAAAAAAAAAAAAAAAAA"
+			"AAAAAAAAAAAAAAAAAAAAAAAAAAAAAAAAAAAAAAAAAAAAAAAAAAAAAAAAAAAAAAAAAAAAAAAAAAAA"
+			"AAAAAAAAAAAAAAAAAAAAAAAAAAAAAAAAAAAAAAAAAAAAAAAAAAAAAAAAAAAAAAAAAAAAAAAAAAAA"
+			"AAAAAAAAAAAAAAAAAAAAAAAAAAAAAAAAAAAAAAAAAAAAAAAAAAAAAAAAAAAAAAAAAAAAAAAAAAAA"
+			"AAAAAAAAAAAAAAAAAAAAAAAAAAAAAAAAAAAAAAAAAAAAAAAAAAAAAAAAAAAAAAAAAAAAAAAAAAAA"
+			"AAAAAAAAAAAAAAAAAAAAAAAAAAAAAAAAAAAAAAAAAAAAAAAAAAAAAAAAAAAAAAAAAAAAAAAAAAAA"
+			"AAAAAAAAAAAAAAAAAAAAAAAAAAAAAAAAAAAAAAAAAAAAAAAAAAAAAAAAAAAAAAAAAAAAAAAAAAAA"
+			"AAAAAAAAAAAAAAAAAAAAAAAAAAAAAAAAAAAAAAAAAAAAAAAAAAAAAAAAAAAAAAAAAAAAAAAAAAAA"
 			"AAAAAAAAAAAAAAAAAAAAAAAAAAAAAAAAAAAAAA=="
 		)
@@
 	)
 	(segment
-		(start 70.785 50.3484)
-		(end 70.785 49.6633)
+		(start 65.8257 57.0157)
+		(end 65.8257 50.2923)
 		(width 0.2)
 		(layer "F.Cu")
@@
 	)
 	(segment
-		(start 68.595 48.5)
-		(end 69.6217 48.5)
+		(start 69.81 61)
+		(end 65.8257 57.0157)
 		(width 0.2)
 		(layer "F.Cu")
@@
 	)
 	(segment
-		(start 70.785 49.6633)
-		(end 69.6217 48.5)
+		(start 65.8257 50.2923)
+		(end 67.618 48.5)
 		(width 0.2)
 		(layer "F.Cu")
 		(net 2)
 	)
-	(via
-		(at 70.785 50.3484)
-		(size 0.6)
-		(drill 0.3)
-		(layers "F.Cu" "B.Cu")
-		(net 2)
-	)
 	(segment
-		(start 68.7622 55.5646)
-		(end 69.3686 54.9582)
+		(start 67.618 48.5)
+		(end 68.595 48.5)
 		(width 0.2)
-		(layer "B.Cu")
-		(net 2)
-	)
-	(segment
-		(start 69.3686 54.9582)
-		(end 69.3686 51.7648)
-		(width 0.2)
-		(layer "B.Cu")
-		(net 2)
-	)
-	(segment
-		(start 68.7622 58.9505)
-		(end 68.7622 55.5646)
-		(width 0.2)
-		(layer "B.Cu")
-		(net 2)
-	)
-	(segment
-		(start 69.81 59.9983)
-		(end 68.7622 58.9505)
-		(width 0.2)
-		(layer "B.Cu")
-		(net 2)
-	)
-	(segment
-		(start 69.81 61)
-		(end 69.81 59.9983)
-		(width 0.2)
-		(layer "B.Cu")
-		(net 2)
-	)
-	(segment
-		(start 69.3686 51.7648)
-		(end 70.785 50.3484)
-		(width 0.2)
-		(layer "B.Cu")
+		(layer "F.Cu")
 		(net 2)
 	)
@@
 		(net 27)
 		(net_name "/GND")
-		(layer "B.Cu")
+		(layers "F.Cu" "B.Cu")
 		(hatch edge 0.5)
 		(connect_pads
