File: cad/stone_pcb_v1.kicad_pcb (KiCad board)
At the start: 2 copper layers, 70.4 x 38.9 mm, 18 parts, among them J10 Conn_01x02_Socket 5V & GND CA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, J2 DRV8833, J3 Conn_01x04_Socket, J6 S2-Mini, J7 Breakouts, J8 S2-Mini, J9 Conn_01x02_Socket EXT_5V & GND, M1 TP Motor1, M2 TP Motor2, M3 TP Motor3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

Commit message: updated pcb
Parts:
- TP7: value Switch1 -> S1
- TP8: value Switch2 -> S2
- renumbered J10 to CAM
Other:
- outline, holes or cut-outs redrawn
- board text added: "| | \ \ | / / \ \ | / / \ \ | / / \ \|/ / *** / /|\ \ / / | \ \ / / | \ \ / / | \ \ | |"
- board text added: "| | | \ \ | / / \ \ | / / \ \ | / / \ \|/ / *** / /|\ \ / / | \ \ / / | \ \ / / | \ \ | | |"
- board text removed: "| | | \ \ | / / \ \ | / / \ \ | / / \ \|/ / ----- *** ----- / /|\ \ / / | \ \ / / | \ \ / / | \ \ | | |"
