File: cad/stone_pcb_v1-2025-04-14_230358/stone_pcb_v1.kicad_pcb (KiCad board)
At the start: 2 copper layers, 70.4 x 38.9 mm, 18 parts, among them J10 Conn_01x02_Socket 5V & GND CA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, J2 DRV8833, J3 Conn_01x04_Socket, J6 S2-Mini, J7 Breakouts, J8 S2-Mini, J9 Conn_01x02_Socket EXT_5V & GND, M1 TP Motor1, M2 TP Motor2, M3 TP Motor3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

Commit message: updated pcb
Parts:
- renumbered M1 to TP1, M2 to TP2, M3 to TP3, M4 to TP4
Other:
- board text added: "(symbol "LOGO" (pin_names (offset 1.016)) (in_bom yes) (on_board yes) (property "Reference" "#G" (at 0 139.78 0) (effects (font (size 1.27 1.27)) hide) ) (property "Value" "LOGO" (at 0 -139.78 0) (effects (font (size 1.27 1.27)) hide) ) (property "Footprint" "" (at 0 0 0) (effects (font (size 1.27 1.27)) hide) ) (property "Datasheet" "" (at 0 0 0) (effects (font (size 1.27 1.27)) hide) ) (symbol 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"
- board text removed: "_ _ __ _ __| |_ | '_ \| '__| __| | |_) | | | |_ | .__/|_| \__| |_|"
- board text removed: "_-._ __./ '\ / '\ '\ /*'-. | | | | \ \.___/_.__./ \_____/"
